Commit message: feat: add adjustable virtual IK tip link

File: src/moveit_whole_body_ik/urdf/ir100.xacro (robot description, xacro)
@@ -52,4 +52,11 @@
             <parent link="Link6" />
             <child link="arm_gripper_link" />
+        </joint>
+        <!-- Virtual IK tool center: 0.14 m along arm_gripper_link local +Z. -->
+        <link name="ik_tip_link" />
+        <joint name="ik_tip_joint" type="fixed">
+            <origin xyz="0 0 0.14" rpy="0 0 0" />
+            <parent link="arm_gripper_link" />
+            <child link="ik_tip_link" />
         </joint>
    <link name="left_wheel_link" />
